File: hardware/main_board/6502_computer.kicad_pcb (KiCad board)
At the start: 2 copper layers, 225.1 x 142 mm, 78 parts, among them J1 Conn_02x20_Odd_Even, J2 Conn_01x40_Socket, J3 Conn_01x40_Socket, J4 Conn_01x02_Pin, J5 RCJ-045, J6 DE9_Pins, J7 Mini-DIN-6, J8 Conn_01x12_Pin, Q1 2SC1815, SW1 SW_Push, U1 6502, U10 74HC138, U11 74HC595, U12 74HC138, U13 6522, U14 74HCT04, U15 MAX232, U16 6551, U17 74HC595, U18 74HC14, U2 74LS574, U3 74LS574, U4 HM62256BLP, U5 74LS574, U6 tms9918, U7 HM62256BLP, U8 74HC00, U9 28C256, Y1 CXO_DIP8, Y2 10.738635Mhz, Y3 1.8432MHz

Commit message: updated pcb and sch
Connections:
- U17 pad 9: /unconnected-(U8-QH&amp;apos;-Pad9) -> unconnected-(U17-QH&apos;-Pad9)
Routing:
- net 1Mhz clk: track 450.2 -> 449.1 mm
Other:
- board text added: "x"
Changed lines of the file:
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@@
 	(net 150 "unconnected-(U17-QH-Pad7)")
 	(net 151 "unconnected-(U17-QC-Pad2)")
-	(net 152 "/unconnected-(U8-QH&amp;apos;-Pad9)")
+	(net 152 "unconnected-(U17-QH&apos;-Pad9)")
 	(net 153 "unconnected-(U17-QF-Pad5)")
 	(net 154 "unconnected-(U17-QE-Pad4)")
@@
 			(layers "*.Cu" "*.Mask")
 			(remove_unused_layers no)
-			(net 152 "/unconnected-(U8-QH&amp;apos;-Pad9)")
+			(net 152 "unconnected-(U17-QH&apos;-Pad9)")
 			(pinfunction "QH'")
 			(pintype "output+no_connect")
@@
 		)
 	)
+	(gr_text "x"
+		(at 188.65 71.6 0)
+		(layer "F.SilkS")
+		(effects
+			(font
+				(size 1 1)
+				(thickness 0.2)
+				(bold yes)
+			)
+			(justify left bottom)
+		)
+	)
 	(gr_text "$C000-$FFFF"
 		(at 201.838095 137.035875 0)
@@
 		)
 	)
+	(gr_text "x"
+		(at 234.15 132.75 0)
+		(layer "F.SilkS")
+		(effects
+			(font
+				(size 1 1)
+				(thickness 0.2)
+				(bold yes)
+			)
+			(justify left bottom)
+		)
+	)
 	(gr_text "PB6"
 		(at 198.206818 150.3 90)
@@
 		)
 	)
+	(gr_text "x"
+		(at 188.45 46.2 0)
+		(layer "F.SilkS")
+		(effects
+			(font
+				(size 1 1)
+				(thickness 0.2)
+				(bold yes)
+			)
+			(justify left bottom)
+		)
+	)
 	(gr_text "$8000-$83FF"
 		(at 201.652382 108.94375 0)
@@
 	)
 	(gr_text "VDD"
-		(at 186.4 74.3 0)
+		(at 186.7 74.3 0)
 		(layer "F.SilkS")
 		(effects
@@
 	)
 	(segment
-		(start 186.8 127.8)
-		(end 187.6 127)
+		(start 184.7 100.88)
+		(end 187.6 103.78)
 		(width 0.3)
 		(layer "F.Cu")
@@
 	)
 	(segment
+		(start 187.6 103.78)
+		(end 187.6 127)
+		(width 0.3)
+		(layer "F.Cu")
+		(net 30)
+	)
+	(segment
 		(start 104.4 48.23)
 		(end 104.4 69.31)
@@
 	)
 	(segment
-		(start 124.34 35.59)
-		(end 113.029 46.901)
+		(start 184.675 64.455)
+		(end 184.7 64.48)
 		(width 0.3)
 		(layer "F.Cu")
@@
 	)
 	(segment
-		(start 97 101.79)
-		(end 97 97.23)
+		(start 124.34 35.59)
+		(end 113.029 46.901)
 		(width 0.3)
 		(layer "F.Cu")
@@
 	)
 	(segment
-		(start 184.675 64.455)
-		(end 183.4 65.73)
+		(start 97 101.79)
+		(end 97 97.23)
 		(width 0.3)
 		(layer "F.Cu")
@@
 	)
 	(segment
-		(start 187.6 103.78)
-		(end 183.4 99.58)
-		(width 0.3)
-		(layer "F.Cu")
-		(net 30)
-	)
-	(segment
 		(start 170.31 132.11)
 		(end 179.89 132.11)
@@
 	)
 	(segment
-		(start 183.4 65.73)
-		(end 183.4 99.58)
+		(start 132.3 124.83)
+		(end 134.4 126.93)
 		(width 0.3)
 		(layer "F.Cu")
@@
 	)
 	(segment
-		(start 132.3 124.83)
-		(end 134.4 126.93)
+		(start 184.2 127.8)
+		(end 179.89 132.11)
 		(width 0.3)
 		(layer "F.Cu")
@@
 	)
 	(segment
-		(start 187.6 127)
-		(end 187.6 103.78)
+		(start 158.95 126.93)
+		(end 160.35 128.33)
 		(width 0.3)
 		(layer "F.Cu")
@@
 	)
 	(segment
-		(start 184.2 127.8)
+		(start 187.6 127)
 		(end 186.8 127.8)
 		(width 0.3)
@@
 	)
 	(segment
-		(start 179.89 132.11)
-		(end 184.2 127.8)
+		(start 105.729 46.901)
+		(end 104.4 48.23)
 		(width 0.3)
 		(layer "F.Cu")
@@
 	)
 	(segment
-		(start 158.95 126.93)
-		(end 160.35 128.33)
+		(start 195.4 64.78)
+		(end 196.658471 64.78)
 		(width 0.3)
 		(layer "F.Cu")
@@
 	)
 	(segment
-		(start 105.729 46.901)
-		(end 104.4 48.23)
+		(start 184.7 64.48)
+		(end 184.7 100.88)
 		(width 0.3)
 		(layer "F.Cu")
@@
 	)
 	(segment
-		(start 195.4 64.78)
-		(end 196.658471 64.78)
+		(start 104.4 69.31)
+		(end 101.2 72.51)
 		(width 0.3)
 		(layer "F.Cu")
@@
 	)
 	(segment
-		(start 104.4 69.31)
-		(end 101.2 72.51)
+		(start 186.8 127.8)
+		(end 184.2 127.8)
 		(width 0.3)
 		(layer "F.Cu")
@@
 	)
 	(segment
-		(start 116.95 57.88)
-		(end 126.54 48.29)
-		(width 0.3)
-		(layer "B.Cu")
-		(net 43)
-	)
-	(segment
-		(start 126.54 48.29)
-		(end 127.2 48.29)
+		(start 187.499 36.929)
+		(end 195.049 36.929)
 		(width 0.3)
 		(layer "B.Cu")
@@
 	)
 	(segment
-		(start 187.499 36.929)
-		(end 195.049 36.929)
+		(start 58.8 122.84)
+		(end 52.07 129.57)
 		(width 0.3)
 		(layer "B.Cu")
@@
 	)
 	(segment
-		(start 58.8 122.84)
-		(end 52.07 129.57)
+		(start 117 91.63)
+		(end 117 57.83)
 		(width 0.3)
 		(layer "B.Cu")
@@
 	)
 	(segment
-		(start 112.08 96.55)
-		(end 116.95 91.68)
-		(width 0.3)
-		(layer "B.Cu")
-		(net 43)
-	)
-	(segment
 		(start 159 34.23)
 		(end 173.1 34.23)
@@
 	)
 	(segment
+		(start 112.08 96.55)
+		(end 117 91.63)
+		(width 0.3)
+		(layer "B.Cu")
+		(net 43)
+	)
+	(segment
 		(start 179.89 35.59)
 		(end 186.16 35.59)
@@
 	)
 	(segment
-		(start 116.95 91.68)
-		(end 116.95 57.88)
+		(start 63.599 102.781)
+		(end 62.175 104.205)
 		(width 0.3)
 		(layer "B.Cu")
@@
 	)
 	(segment
-		(start 63.599 102.781)
-		(end 62.175 104.205)
+		(start 126.54 48.29)
+		(end 127.2 48.29)
+		(width 0.3)
+		(layer "B.Cu")
+		(net 43)
+	)
+	(segment
+		(start 117 57.83)
+		(end 126.54 48.29)
 		(width 0.3)
 		(layer "B.Cu")
