File: hardware/main_board/6502_computer.kicad_sch (KiCad schematic)
At the start: 54 parts, among them J1 Conn_02x20_Odd_Even, J2 Conn_01x40_Socket, J3 Conn_01x40_Socket, J4 Conn_01x02_Pin, J6 DE9_Pins, J7 Mini-DIN-6, J8 Conn_01x12_Pin, SW1 SW_Push, U1 6502, U11 74HC595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

Commit message: updated pcb and sch
Connections:
- net unconnected-(U8-QH&apos;-Pad9): no longer names the net of U17.9 (QH')
Changed lines of the file:
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@@
-		)
-	)
-	(label "unconnected-(U8-QH&apos;-Pad9)"
-		(at 280.67 156.21 0)
-		(effects
-			(font
-				(size 1.27 1.27)
-			)
-			(justify left bottom)
 		)
 	)
