File: hardware/main_board/video.kicad_sch (KiCad schematic)
At the start: 22 parts, among them J5 RCJ-045, Q1 2SC1815, U10 74HC138, U14 74HCT04, U2 74LS574, U3 74LS574, U5 74LS574, U6 tms9918, U7 HM62256BLP, Y2 10.738635Mhz

Commit message: Adds stuff
Connections:
- net GND: now also J5.1; no longer J5.2
- net VID: now also J5.2; no longer J5.1
Other:
- moved on the sheet: J5
Changed lines of the file:
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@@
 	)
 	(junction
+		(at 72.39 163.83)
+		(diameter 0)
+		(color 0 0 0 0)
+	)
+	(junction
 		(at 74.93 54.61)
 		(diameter 0)
@@
 	)
 	(junction
-		(at 72.39 163.83)
-		(diameter 0)
-		(color 0 0 0 0)
-	)
-	(junction
 		(at 184.15 49.53)
 		(diameter 0)
@@
 	(wire
 		(pts
+			(xy 72.39 163.83) (xy 87.63 163.83)
+		)
+		(stroke
+			(width 0)
+			(type default)
+		)
+	)
+	(wire
+		(pts
 			(xy 160.02 92.71) (xy 166.37 92.71)
 		)
@@
 	(wire
 		(pts
+			(xy 80.01 158.75) (xy 87.63 158.75)
+		)
+		(stroke
+			(width 0)
+			(type default)
+		)
+	)
+	(wire
+		(pts
 			(xy 167.64 69.85) (xy 167.64 67.31)
 		)
@@
 		)
 	)
-	(wire
-		(pts
-			(xy 72.39 163.83) (xy 87.63 163.83)
-		)
-		(stroke
-			(width 0)
-			(type default)
-		)
-	)
 	(bus
 		(pts
@@
 		)
 	)
-	(wire
-		(pts
-			(xy 80.01 158.75) (xy 87.63 158.75)
-		)
-		(stroke
-			(width 0)
-			(type default)
-		)
-	)
 	(bus
 		(pts
@@
 	(symbol
 		(lib_id "RCJ-045:RCJ-045")
-		(at 92.71 161.29 180)
+		(at 92.71 161.29 0)
+		(mirror y)
 		(unit 1)
 		(exclude_from_sim no)
@@
 		(on_board yes)
 		(dnp no)
-		(fields_autoplaced yes)
 		(property "Reference" "J5"
-			(at 100.33 160.0199 0)
+			(at 100.33 162.5601 0)
 			(effects
 				(font
@@
 		)
 		(property "Value" "RCJ-045"
-			(at 100.33 162.5599 0)
+			(at 100.33 160.0201 0)
 			(effects
 				(font

Commit message: updated readme
Parts:
- R4, R5: footprint Resistor_THT:R_Axial_DIN0207_L6.3mm_D2.5mm_P7.62mm_Horizontal -> Resistor_THT:R_Axial_DIN0207_L6.3mm_D2.5mm_P10.16mm_Horizontal
Other:
- note removed: "might need delay here ?"
Changed lines of the file:
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@@
 		)
 	)
-	(text "might need delay here ?\n"
-		(exclude_from_sim no)
-		(at 93.472 85.344 0)
-		(effects
-			(font
-				(size 1.27 1.27)
-			)
-		)
-	)
 	(junction
 		(at 181.61 52.07)
@@
 			)
 		)
-		(property "Footprint" "Resistor_THT:R_Axial_DIN0207_L6.3mm_D2.5mm_P7.62mm_Horizontal"
+		(property "Footprint" "Resistor_THT:R_Axial_DIN0207_L6.3mm_D2.5mm_P10.16mm_Horizontal"
 			(at 61.722 160.02 90)
 			(effects
@@
 			)
 		)
-		(property "Footprint" "Resistor_THT:R_Axial_DIN0207_L6.3mm_D2.5mm_P7.62mm_Horizontal"
+		(property "Footprint" "Resistor_THT:R_Axial_DIN0207_L6.3mm_D2.5mm_P10.16mm_Horizontal"
 			(at 70.612 160.02 90)
 			(effects
